File: cbEval.Busses.kicad_sch (KiCad schematic)
At the start: 25 parts, among them J1 Bergstik-II_3, J2 Bergstik-II_3, J3 Header.Hor.2x8.9-103326-0-08, J4 Header.Hor.2x8.9-103326-0-08, J5 Socket.Hor.2x8.1-5535512-8, J6 Bergstik-II_3, J7 Bergstik-II_6, J8 Bergstik-II_3, J9 Socket.Hor.2x8.1-5535512-8

Commit message: Zwischenstand (Sicherung)
Parts:
- removed J2: Bergstik-II_3, Connector_PinHeader_2.54mm:PinHeader_1x03_P2.54mm_Vertical, symbol J.PinHeader:Bergstik-II_3
- removed J7: Bergstik-II_6, Connector_PinHeader_2.54mm:PinHeader_1x06_P2.54mm_Vertical, symbol J.PinHeader:Bergstik-II_6
- added J19: Bergstik-II_3, Connector_PinHeader_2.54mm:PinHeader_1x03_P2.54mm_Vertical, symbol J.PinHeader:Bergstik-II_3
- added J24: Bergstik-II_6, Connector_PinHeader_2.54mm:PinHeader_1x06_P2.54mm_Vertical, symbol J.PinHeader:Bergstik-II_6
Connections:
- net GND: now also J24.5 (A5)
- net One-Wire: now also J24.6 (A6)
- net SPI-ADR0: now also J19.1 (A1)
- net SPI-ADR1: now also J19.2 (A2)
- net SPI-ADR2: now also J19.3 (A3)
- net SPI-CLK: now also J24.3 (A3)
- net SPI-MRST: now also J24.2 (A2)
- net SPI-MTSR: now also J24.1 (A1)
- net SPI-~{CE}: now also J24.4 (A4)
