File: cbEval.STM32G0B1KET6.kicad_pcb (KiCad board)
At the start: 4 copper layers, 35 x 108 mm, 60 parts, among them J1 Bergstik-II_3, J10 Bergstik-II_6, J11 Bergstik-II_6, J12 Bergstik-II_8, J13 Bergstik-II_6, J14 CNC-Tech 2x5, J15 Bergstik-II_6, J2 Bergstik-II_3, J20 Bergstik-II_3, J21 Bergstik-II_3, J22 Bergstik-II_2, J23 Bergstik-II_2, J3 Header.Hor.2x8.9-103326-0-08, J4 Header.Hor.2x8.9-103326-0-08, J5 Socket.Hor.2x8.1-5535512-8, J6 Bergstik-II_3, J7 Bergstik-II_6, J8 Bergstik-II_3, J9 Socket.Hor.2x8.1-5535512-8, U1 STM32G0B1KET6, Y1 16.000MHz

Commit message: Zwischenstand (Sicherung)
Parts:
- added C10: 1µ(16V), Capacitor_SMD:C_0805_2012Metric, F.Cu at (199.4, 109.9)
- added C11: 1µ(16V), Capacitor_SMD:C_0805_2012Metric, F.Cu at (199.4, 118.8)
- added C12: 1µ(16V), Capacitor_SMD:C_0805_2012Metric, F.Cu at (199.4, 114.3)
- added C13: 1µ(16V), Capacitor_SMD:C_0805_2012Metric, F.Cu at (184.4, 72.4)
- added C14: 100n, Capacitor_SMD:C_0805_2012Metric, F.Cu at (204.7, 118.8)
- added C15: 100n, Capacitor_SMD:C_0805_2012Metric, F.Cu at (221.6, 76.2)
- added C16: 33p, Capacitor_SMD:C_0805_2012Metric, F.Cu at (215.3, 101.0)
- added C7: 100n, Capacitor_SMD:C_0805_2012Metric, F.Cu at (178.1, 106.7)
- added C8: 4µ7, Capacitor_SMD:C_0805_2012Metric, F.Cu at (172.7, 86.4)
- added C9: 100n, Capacitor_SMD:C_0805_2012Metric, F.Cu at (175.3, 89.5)
- added D2: Würth.VS, LED_SMD:LED_0805_2012Metric, F.Cu at (186.7, 63.5)
- added D3: Würth.VS, LED_SMD:LED_0805_2012Metric, F.Cu at (186.7, 60.5)
- added D4: Würth.SS, LED_SMD:LED_0805_2012Metric, F.Cu at (213.2, 65.0)
- added D5: Würth.SS, LED_SMD:LED_0805_2012Metric, F.Cu at (214.5, 61.1)
- added D6: Würth.VS, LED_SMD:LED_0805_2012Metric, F.Cu at (218.9, 61.1)
- added D7: Würth.VS, LED_SMD:LED_0805_2012Metric, F.Cu at (213.2, 68.1)
- added D8: Würth.AS, LED_SMD:LED_0805_2012Metric, F.Cu at (208.7, 65.0)
- added D9: Würth.AS, LED_SMD:LED_0805_2012Metric, F.Cu at (208.7, 68.1)
- added FID1: 1-2mm, Fiducial:Fiducial_1mm_Mask2mm, F.Cu at (153.7, 58.4)
- added FID2: 1-2mm, Fiducial:Fiducial_1mm_Mask2mm, F.Cu at (150.1, 58.4)
- added FID3: 1-2mm, Fiducial:Fiducial_1mm_Mask2mm, F.Cu at (153.7, 54.9)
- added FID4: 1-2mm, Fiducial:Fiducial_1mm_Mask2mm, F.Cu at (150.1, 54.9)
- added J16: Bergstik-II_2x4, Connector_PinHeader_2.54mm:PinHeader_2x04_P2.54mm_Vertical, F.Cu at (168.9, 115.6)
- added J17: Bergstik-II_2x4, Connector_PinHeader_2.54mm:PinHeader_2x04_P2.54mm_Vertical, F.Cu at (159.4, 132.1)
- added J18: Bergstik-II_2x2, Connector_PinHeader_2.54mm:PinHeader_2x02_P2.54mm_Vertical, F.Cu at (141.6, 73.7)
- added J19: Bergstik-II_3, Connector_PinHeader_2.54mm:PinHeader_1x03_P2.54mm_Vertical, F.Cu at (123.8, 55.9)
- added J24: Bergstik-II_6, Connector_PinHeader_2.54mm:PinHeader_1x06_P2.54mm_Vertical, F.Cu at (130.2, 54.6)
- added J25: STD.9P.FEM.Vert.Screw, BTech.Connector.DSub:DSUB-9_Female_Vertical_Harting0966151X51X, F.Cu at (127.0, 135.3)
- added J26: Bergstik-II_2x4, Connector_PinHeader_2.54mm:PinHeader_2x04_P2.54mm_Vertical, F.Cu at (233.4, 61.9)
- added MP1: KiCAD-DesignedWith-Logo2.5mm.SilkScreen, Symbol:KiCad-Logo2_5mm_SilkScreen, F.Cu at (163.2, 55.9)
- added R17: 1k, Resistor_SMD:R_0805_2012Metric, F.Cu at (191.1, 60.4)
- added R18: 1k, Resistor_SMD:R_0805_2012Metric, F.Cu at (191.1, 63.4)
- added R19: 1k, Resistor_SMD:R_0805_2012Metric, F.Cu at (217.6, 64.1)
- added R20: 1k, Resistor_SMD:R_0805_2012Metric, F.Cu at (217.6, 70.0)
- added R21: 1k, Resistor_SMD:R_0805_2012Metric, F.Cu at (222.0, 67.0)
- added R22: 1k, Resistor_SMD:R_0805_2012Metric, F.Cu at (222.0, 64.1)
- added R23: 1k, Resistor_SMD:R_0805_2012Metric, F.Cu at (223.3, 61.0)
- added R24: 1k, Resistor_SMD:R_0805_2012Metric, F.Cu at (217.6, 67.0)
- added R25: 4k7, Resistor_SMD:R_0805_2012Metric, F.Cu at (240.5, 64.0)
- added R26: 4k7, Resistor_SMD:R_0805_2012Metric, F.Cu at (240.5, 61.0)
- added R27: 4k7, Resistor_SMD:R_0805_2012Metric, F.Cu at (244.9, 61.0)
- added R28: 3k9, Resistor_SMD:R_0805_2012Metric, F.Cu at (215.2, 103.9)
- added S5: TL3305A, Button_Switch_SMD:SW_SPST_TL3305A, F.Cu at (173.4, 81.3)
- added TP6: SMT5019, TestPoint:TestPoint_Keystone_5019_Minature, F.Cu at (209.4, 61.5)
- added TP7: SMT5019, TestPoint:TestPoint_Keystone_5019_Minature, F.Cu at (210.2, 101.4)
- added U2: TRSF3238EIDWR, Package_SO:SOIC-28W_7.5x18.7mm_P1.27mm, F.Cu at (193.1, 81.1)
- added U3: MCP23016-I/SO, Package_SO:SOIC-28W_7.5x18.7mm_P1.27mm, F.Cu at (212.1, 82.5)
- H1: value CIME.E.BE3500S.1x -> CIME.E.BE3500S.2x; footprint BTech.Housing:Camdenboss.CIME.E.BE3500S.1x -> BTech.PCB:Camdenboss.CIME.E.BE3500S.2x
- J2: value Bergstik-II_3 -> Bergstik-II_2x4; footprint Connector_PinHeader_2.54mm:PinHeader_1x03_P2.54mm_Vertical -> Connector_PinHeader_2.54mm:PinHeader_2x04_P2.54mm_Vertical
- J7: value Bergstik-II_6 -> Bergstik-II_2x4; footprint Connector_PinHeader_2.54mm:PinHeader_1x06_P2.54mm_Vertical -> Connector_PinHeader_2.54mm:PinHeader_2x04_P2.54mm_Vertical
- R7: value 649R -> 680R
- moved J11 61.8 mm to (122.6, 87.6)
- moved J13 60.6 mm to (122.6, 107.3)
- moved J12 60.3 mm to (117.5, 83.2)
- moved J10 56.9 mm to (116.8, 108.6)
- moved J2 55.7 mm to (175.9, 114.9), turned to 0 degrees
- moved JP5 52.2 mm to (122.6, 74.9)
- moved JP4 20.5 mm to (165.7, 74.9)
- moved J3 17.8 mm to (116.1, 149.2)
- moved J4 17.8 mm to (116.1, 70.5)
- moved J5 17.5 mm to (179.4, 62.9)
- moved J9 17.5 mm to (179.4, 141.6)
- moved C6 8.45 mm to (177.5, 100.3)
- moved J7 3.82 mm to (145.4, 116.2)
Connections:
- net Net-(J10-Pad3) renamed /MCU/PA15
- net Net-(J10-Pad4) renamed /MCU/PB3
- net Net-(J10-Pad5) renamed /MCU/PB4
- net Net-(J10-Pad6) renamed /MCU/PB5
- net Net-(J11-Pad1) renamed /MCU/PB6
- net Net-(J11-Pad2) renamed /MCU/PB7
- net Net-(J12-Pad5) renamed /MCU/PA4
- net Net-(J12-Pad7) renamed /MCU/PA6
- net Net-(J12-Pad8) renamed /MCU/PA7
- net Net-(J13-Pad1) renamed /MCU/PA8
- net Net-(J13-Pad2) renamed /MCU/PA9
- net Net-(J13-Pad3) renamed /MCU/PA10
- net Net-(J13-Pad4) renamed /MCU/PA11
- net Net-(J13-Pad5) renamed /MCU/PA12
- net Net-(J13-Pad6) renamed /MCU/PB2
- net Net-(U1-Pad12) renamed /MCU/PA5
- J10 pad 1: Net-(J10-Pad1) -> /MCU/PA13
- J10 pad 2: Net-(J10-Pad2) -> /MCU/PA14
- J11 pad 3: Net-(J11-Pad3) -> /MCU/PB8
- J11 pad 4: Net-(J11-Pad4) -> /MCU/PB9
- J11 pad 5: Net-(J11-Pad5) -> /MCU/PB0
- J11 pad 6: Net-(J11-Pad6) -> /MCU/PB1
- J12 pad 1: Net-(J12-Pad1) -> /MCU/PA0
- J12 pad 2: Net-(J12-Pad2) -> /MCU/PA1
- J12 pad 3: Net-(J12-Pad3) -> /MCU/PA2
- J12 pad 4: Net-(J12-Pad4) -> /MCU/PA3
- J14 pad 1: unconnected-(J14-Pad1) -> PwrMCU
- J14 pad 10: unconnected-(J14-Pad10) -> /MCU/PF2
- J14 pad 2: unconnected-(J14-Pad2) -> /MCU/PA13
- J14 pad 3: unconnected-(J14-Pad3) -> GND
- J14 pad 4: unconnected-(J14-Pad4) -> /MCU/PA14
- J14 pad 5: unconnected-(J14-Pad5) -> GND
- J14 pad 9: unconnected-(J14-Pad9) -> GND
- J2 pad 1: /Busses/SPI-ADR0 -> /MCU/PA2
- J2 pad 2: /Busses/SPI-ADR1 -> /MCU/UART-Tx
- J2 pad 3: /Busses/SPI-ADR2 -> /MCU/PA3
- J7 pad 1: /Busses/SPI-MTSR -> /MCU/CAN1-Rx
- J7 pad 2: /Busses/SPI-MRST -> /MCU/PB8
- J7 pad 3: /Busses/SPI-CLK -> /MCU/CAN1-Tx
- J7 pad 4: /Busses/SPI-~{CE} -> /MCU/PB9
- J7 pad 5: GND -> /MCU/CAN2-Rx
- J7 pad 6: /Busses/One-Wire -> /MCU/PB0
- JP2 pad 2: VCC -> PwrMCU
- TP3 pad 1: VCC -> PwrMCU
- U1 pad 1: Net-(J11-Pad4) -> /MCU/PB9
- U1 pad 10: Net-(J12-Pad4) -> /MCU/PA3
- U1 pad 15: Net-(J11-Pad5) -> /MCU/PB0
- U1 pad 16: Net-(J11-Pad6) -> /MCU/PB1
- U1 pad 20: (no net) -> /MCU/PC6
- U1 pad 24: Net-(J10-Pad1) -> /MCU/PA13
- U1 pad 25: Net-(J10-Pad2) -> /MCU/PA14
- U1 pad 32: Net-(J11-Pad3) -> /MCU/PB8
- U1 pad 6: unconnected-(U1-Pad6) -> /MCU/PF2
- U1 pad 7: Net-(J12-Pad1) -> /MCU/PA0
- U1 pad 8: Net-(J12-Pad2) -> /MCU/PA1
- U1 pad 9: Net-(J12-Pad3) -> /MCU/PA2
Other:
- board size 35 x 108 mm -> 70 x 108 mm
