File: cbEval.STM32G0B1KET6.kicad_sch (KiCad schematic)
At the start: 15 parts, among them J15 Bergstik-II_6, J20 Bergstik-II_3, J21 Bergstik-II_3, J22 Bergstik-II_2, J23 Bergstik-II_2

Commit message: Zwischenstand (Sicherung)
Parts:
- removed H1: CIME.E.BE3500S.1x, BTech.Housing:Camdenboss.CIME.E.BE3500S.1x, symbol H.Housing:CIME.E.BE3500S.1x
- added FID1, FID2, FID3, FID4: 1-2mm, Fiducial:Fiducial_1mm_Mask2mm, symbol FID:1-2mm
- added H1: CIME.E.BE3500S.2x, BTech.PCB:Camdenboss.CIME.E.BE3500S.2x, symbol H.Housing:CIME.E.BE3500S.2x
- added MP1: KiCAD-DesignedWith-Logo2.5mm.SilkScreen, Symbol:KiCad-Logo2_5mm_SilkScreen, symbol Symbol:KiCAD-DesignedWith-Logo2.5mm.SilkScreen
- R7: value 649R -> 680R; symbol R.Yageo.RC0805:649R -> R.Yageo.RC0805:680R; ID RC0805FR-07649RL -> RC0805FR-07680RL
Other:
- added sheet CAN-FD Transceiver (CAN-FD-Transceiver.kicad_sch)
- added sheet Port Extension I2C (PortExtension.I2C.kicad_sch)
- added sheet RS-232 Transceiver (RS-232_5-3.kicad_sch)
- sheet Busses ports: added I2C-SCL, I2C-SDA, One-Wire, SPI-ADR0, SPI-ADR1, SPI-ADR2, SPI-CLK, SPI-MRST, SPI-MTSR, SPI-~{CE}, ~{RESET}; removed none
- sheet MCU ports: added CAN1-Rx, CAN1-Tx, CAN2-Rx, CAN2-Tx, I2C-Aux-SCL, I2C-Aux-SDA, I2C-Aux-~{INT}, I2C-SCL, I2C-SDA, PwrMCU, SPI-ADR0, SPI-ADR1, SPI-ADR2, SPI-CLK, SPI-MRST, SPI-MTSR, SPI-~{CE}, UART-CTS, UART-RTS, UART-Rx, UART-Tx; removed none
- title: cbEval ATtiny412 & ATtiny1614 -> cbEval STM32G0B1
- moved on the sheet: D1A, D1B, J15, J20, J21, J22, J23, R5, R6, R7, R8, S3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
